Commit message: first commit

File: src/robile_robot/urdf/robile_robot2.urdf (robot description, URDF)
Before this commit: robot ugv_robot, 7 links, 6 joints
Links:
- link base_link: geometry collision box size=0.5 0.3 0.2; visual box size=0.5 0.3 0.2
Joints:
- joint scan_joint: origin xyz=0 0 0 rpy=0 0 0 -> xyz=0 0 0.3 rpy=0 0 0
