Commit message: Initial commit - add URDF file

File: src/robile_robot/urdf/robile_robot.urdf (robot description, URDF)
Before this commit: robot ugv_robot, 5 links, 4 joints
Links:
- link base_link: geometry collision mesh filename=package://robile_robot/models/than.stl; visual mesh filename=package://robile_robot/models/than.stl

File: src/robile_robot/urdf/save.urdf (robot description, URDF)
Before this commit: robot mobile_robot, 5 links, 4 joints
Links:
- removed link rear_left_wheel
- added link near_left_wheel; visual cylinder length=0.05 radius=0.05
Joints:
- removed joint front_right_wheel_joint
- removed joint rear_left_wheel_joint
- added joint near_left_wheel_joint: type continuous, parent base_link, child near_left_wheel, origin xyz=0.18 0.2 -0.01 rpy=0 1.57 0, axis 0 1 0
- added joint rear_front_wheel_joint: type continuous, parent base_link, child front_right_wheel, origin xyz=-0.18 -0.1 -0.01 rpy=0 1.57 0, axis 0 1 0
- joint front_left_wheel_joint: origin xyz=0.18 0.2 -0.01 rpy=0 1.57 0 -> xyz=0.18 -0.1 -0.01 rpy=0 1.57 0
- joint rear_right_wheel_joint: origin xyz=-0.18 -0.1 -0.01 rpy=0 1.57 0 -> xyz=-0.18 0.2 -0.01 rpy=0 1.57 0

Commit message: Initial commit

File: src/robile_robot/urdf/robile_robot.urdf (robot description, URDF)
Before this commit: robot ugv_robot, 7 links, 6 joints
Links:
- added link tower_scan, mass 0.114; collision cylinder length=0.3 radius=0.02; visual cylinder length=0.3 radius=0.02
Joints:
- added joint tower_joint: type fixed, parent base_link, child tower_scan, origin xyz=0.35 0.0 0.33 rpy=0.0 0.0 0.0
- joint joint_wheel_ph_s: origin xyz=0.2 -0.16 -0.1 rpy=1.57 0.0 0.0 -> xyz=0.2 0.16 -0.1 rpy=1.57 0.0 0.0
- joint joint_wheel_ph_trc: origin xyz=0.2 0.16 -0.1 rpy=1.57 0.0 0.0 -> xyz=-0.2 0.16 -0.1 rpy=1.57 0.0 0.0
- joint joint_wheel_tr_s: origin xyz=-0.2 -0.16 -0.1 rpy=1.57 0.0 0.0 -> xyz=0.2 -0.16 -0.1 rpy=1.57 0.0 0.0
- joint joint_wheel_tr_trc: origin xyz=-0.2 0.16 -0.1 rpy=1.57 0.0 0.0 -> xyz=-0.2 -0.16 -0.1 rpy=1.57 0.0 0.0
- joint scan_joint: origin xyz=0 0 0 rpy=0 0 0 -> xyz=0.35 0 0.5 rpy=0 0 0

Commit message: first commit

File: src/robile_robot/urdf/robile_robot.urdf (robot description, URDF)
Before this commit: robot ugv_robot, 7 links, 6 joints
Links:
- link base_link: geometry collision mesh filename=package://robile_robot/models/body5.stl; visual mesh filename=package://robile_robot/models/body5.stl

File: src/robile_robot/xacro/robile_robot_ur5.xacro (robot description, xacro)
@@ -7,5 +7,5 @@
     <visual>
       <geometry>
-        <mesh filename="package://robile_robot/models/body3.stl"/>
+        <mesh filename="package://robile_robot/models/body5.stl"/>
       </geometry>
       <material name="pink">
@@ -16,5 +16,5 @@
     <collision>
       <geometry>
-        <mesh filename="package://robile_robot/models/body3.stl"/>
+        <mesh filename="package://robile_robot/models/body5.stl"/>
       </geometry>
     </collision>
