Commit message: first commit

File: src/robile_robot/urdf/robile_robot 1.urdf (robot description, URDF)
Before this commit: robot mobile_robot, 5 links, 4 joints
Links:
- removed link front_left_wheel
- removed link front_right_wheel
- removed link rear_left_wheel
- removed link rear_right_wheel
- added link cube, mass 1.0; collision box size=0.2 0.2 0.5; visual box size=0.2 0.2 0.5
- added link wheel_ph_trc, mass 0.5; collision cylinder length=0.1 radius=0.4; visual cylinder length=0.1 radius=0.4
- added link wheel_tr_trc, mass 0.5; collision cylinder length=0.1 radius=0.4; visual cylinder length=0.1 radius=0.4
- link base_link: mass 5 -> 2.0; geometry collision box size=0.5 0.3 0.1; visual box size=0.5 0.3 0.1
Joints:
- removed joint front_left_wheel_joint
- removed joint front_right_wheel_joint
- removed joint rear_left_wheel_joint
- removed joint rear_right_wheel_joint
- added joint joint_cube: type fixed, parent base_link, child cube, origin xyz=0 0 0.3 rpy=0 0 0
- added joint joint_wheel_ph_trc: type continuous, parent base_link, child wheel_ph_trc, origin xyz=0 0.2465 0 rpy=1.5708 0 0, axis 0 1 0
- added joint joint_wheel_tr_trc: type continuous, parent base_link, child wheel_tr_trc, origin xyz=0 -0.2465 0 rpy=1.5708 0 0, axis 0 1 0

File: src/robile_robot/urdf/robile_robot.urdf (robot description, URDF)
Before this commit: robot ugv_robot, 8 links, 7 joints
Links:
- removed link tower_scan
- link base_link: mass 5 -> 2; geometry collision mesh filename=package://robile_robot/models/body3.stl; visual mesh filename=package://robile_robot/models/body3.stl
- link base_scan: mass 0.114 -> 0.1; geometry collision cylinder length=0.1 radius=0.1; visual cylinder length=0.1 radius=0.1
- link camera_link: geometry visual mesh filename=package://robile_robot/models/eye.stl scale=0.5 0.5 0.5
- link wheel_ph_s: mass 10 -> 1; geometry collision cylinder length=0.2 radius=0.2; visual cylinder length=0.2 radius=0.2
- link wheel_ph_trc: mass 10 -> 1; geometry collision cylinder length=0.2 radius=0.2; visual cylinder length=0.2 radius=0.2
- link wheel_tr_s: mass 10 -> 1; geometry collision cylinder length=0.2 radius=0.2; visual cylinder length=0.2 radius=0.2
- link wheel_tr_trc: mass 10 -> 1; geometry collision cylinder length=0.2 radius=0.2; visual cylinder length=0.2 radius=0.2
Joints:
- removed joint tower_joint
- joint camera_joint: origin xyz=-0.15 0.0 0.12 rpy=0 0 3.14 -> xyz=-0.15 -0.40 1.45 rpy=0 0 3.14
- joint joint_wheel_ph_s: origin xyz=0.2 0.16 -0.1 rpy=1.57 0.0 0.0 -> xyz=0.7 0.6 0.2 rpy=1.57 0 0
- joint joint_wheel_ph_trc: origin xyz=-0.2 0.16 -0.1 rpy=1.57 0.0 0.0 -> xyz=-0.3 0.6 0.2 rpy=1.57 0 0
- joint joint_wheel_tr_s: origin xyz=0.2 -0.16 -0.1 rpy=1.57 0.0 0.0 -> xyz=0.7 -0.865 0.2 rpy=1.57 0 0
- joint joint_wheel_tr_trc: origin xyz=-0.2 -0.16 -0.1 rpy=1.57 0.0 0.0 -> xyz=-0.3 -0.865 0.2 rpy=1.57 0 0
- joint scan_joint: origin xyz=0.35 0 0.5 rpy=0 0 0 -> xyz=0 -0.17 1.57 rpy=0 0 0

File: src/robile_robot/urdf/robile_robot2.urdf (robot description, URDF)
Before this commit: robot ugv_robot, 7 links, 6 joints
Links:
- added link tower_scan, mass 0.114; collision cylinder length=0.3 radius=0.02; visual cylinder length=0.3 radius=0.02
- link base_link: geometry collision mesh filename=package://robile_robot/models/than.stl; visual mesh filename=package://robile_robot/models/than.stl
Joints:
- added joint tower_joint: type fixed, parent base_link, child tower_scan, origin xyz=0.35 0.0 0.33 rpy=0.0 0.0 0.0
- joint joint_wheel_ph_s: origin xyz=0.2 -0.16 -0.1 rpy=1.57 0.0 0.0 -> xyz=0.2 0.16 -0.1 rpy=1.57 0.0 0.0
- joint joint_wheel_ph_trc: origin xyz=0.2 0.16 -0.1 rpy=1.57 0.0 0.0 -> xyz=-0.2 0.16 -0.1 rpy=1.57 0.0 0.0
- joint joint_wheel_tr_s: origin xyz=-0.2 -0.16 -0.1 rpy=1.57 0.0 0.0 -> xyz=0.2 -0.16 -0.1 rpy=1.57 0.0 0.0
- joint joint_wheel_tr_trc: origin xyz=-0.2 0.16 -0.1 rpy=1.57 0.0 0.0 -> xyz=-0.2 -0.16 -0.1 rpy=1.57 0.0 0.0
- joint scan_joint: origin xyz=0 0 0.3 rpy=0 0 0 -> xyz=0.35 0 0.5 rpy=0 0 0

File: src/robile_robot/urdf/save.urdf (robot description, URDF)
Before this commit: robot mobile_robot, 5 links, 4 joints
Links:
- removed link front_left_wheel
- removed link front_right_wheel
- removed link near_left_wheel
- removed link rear_right_wheel
- added link base_scan, mass 0.1; collision cylinder length=0.1 radius=0.1; visual cylinder length=0.1 radius=0.1
- added link camera_link, mass 0.1; visual mesh filename=package://robile_robot/models/eye.stl scale=0.5 0.5 0.5
- added link wheel_ph_s, mass 1; collision cylinder length=0.2 radius=0.2; visual cylinder length=0.2 radius=0.2
- added link wheel_ph_trc, mass 1; collision cylinder length=0.2 radius=0.2; visual cylinder length=0.2 radius=0.2
- added link wheel_tr_s, mass 1; collision cylinder length=0.2 radius=0.2; visual cylinder length=0.2 radius=0.2
- added link wheel_tr_trc, mass 1; collision cylinder length=0.2 radius=0.2; visual cylinder length=0.2 radius=0.2
- link base_link: mass None -> 2; geometry collision mesh filename=package://robile_robot/models/body3.stl; visual mesh filename=package://robile_robot/models/body3.stl
Joints:
- removed joint front_left_wheel_joint
- removed joint near_left_wheel_joint
- removed joint rear_front_wheel_joint
- removed joint rear_right_wheel_joint
- added joint camera_joint: type fixed, parent base_link, child camera_link, origin xyz=0 0 1.45 rpy=0 0 3.14
- added joint joint_wheel_ph_s: type continuous, parent base_link, child wheel_ph_s, origin xyz=0.7 0.6 0.2 rpy=1.57 0 0, axis 0 0 1
- added joint joint_wheel_ph_trc: type continuous, parent base_link, child wheel_ph_trc, origin xyz=-0.3 0.6 0.2 rpy=1.57 0 0, axis 0 0 1
- added joint joint_wheel_tr_s: type continuous, parent base_link, child wheel_tr_s, origin xyz=0.7 -0.865 0.2 rpy=1.57 0 0, axis 0 0 1
- added joint joint_wheel_tr_trc: type continuous, parent base_link, child wheel_tr_trc, origin xyz=-0.3 -0.865 0.2 rpy=1.57 0 0, axis 0 0 1
- added joint scan_joint: type fixed, parent base_link, child base_scan, origin xyz=0 -0.17 1.57 rpy=0 0 0

Commit message: first commit

File: src/robile_robot/urdf/robile_robot 1.urdf (robot description, URDF)
Before this commit: robot robile_robot, 4 links, 3 joints
Links:
- removed link cube
- added link base_scan, mass 0.1; collision cylinder length=0.1 radius=0.1; visual cylinder length=0.1 radius=0.1
- added link camera_link, mass 0.1; visual mesh filename=package://robile_robot/models/eye.stl scale=0.5 0.5 0.5
- added link wheel_ph_s, mass 1; collision cylinder length=0.2 radius=0.2; visual cylinder length=0.2 radius=0.2
- added link wheel_tr_s, mass 1; collision cylinder length=0.2 radius=0.2; visual cylinder length=0.2 radius=0.2
- link base_link: mass 2.0 -> 2; geometry collision mesh filename=package://robile_robot/models/body5.stl; visual mesh filename=package://robile_robot/models/body5.stl
- link wheel_ph_trc: mass 0.5 -> 1; geometry collision cylinder length=0.2 radius=0.2; visual cylinder length=0.2 radius=0.2
- link wheel_tr_trc: mass 0.5 -> 1; geometry collision cylinder length=0.2 radius=0.2; visual cylinder length=0.2 radius=0.2
Joints:
- removed joint joint_cube
- added joint camera_joint: type fixed, parent base_link, child camera_link, origin xyz=-0.15 -0.40 1.45 rpy=0 0 3.14
- added joint joint_wheel_ph_s: type continuous, parent base_link, child wheel_ph_s, origin xyz=0.7 0.6 0.2 rpy=1.57 0 0, axis 0 0 1
- added joint joint_wheel_tr_s: type continuous, parent base_link, child wheel_tr_s, origin xyz=0.7 -0.865 0.2 rpy=1.57 0 0, axis 0 0 1
- added joint scan_joint: type fixed, parent base_link, child base_scan, origin xyz=0 -0.17 1.57 rpy=0 0 0
- joint joint_wheel_ph_trc: axis 0 1 0 -> 0 0 1; origin xyz=0 0.2465 0 rpy=1.5708 0 0 -> xyz=-0.3 0.6 0.2 rpy=1.57 0 0
- joint joint_wheel_tr_trc: axis 0 1 0 -> 0 0 1; origin xyz=0 -0.2465 0 rpy=1.5708 0 0 -> xyz=-0.3 -0.865 0.2 rpy=1.57 0 0

File: src/robile_robot/urdf/robile_robot.urdf (robot description, URDF)
Before this commit: robot ugv_robot, 7 links, 6 joints
Links:
- added link base_camera, mass 0.4; visual mesh filename=package://robile_robot/models/eye4.stl
- link camera_link: mass 0.1 -> 0.2; geometry visual cylinder length=0.05 radius=0.07
Joints:
- added joint base_camera_joint: type fixed, parent base_link, child base_camera, origin xyz=0 -0.65 1.115 rpy=0 0 0
- joint camera_joint: axis (none) -> 0.0 0.0 0.0; origin xyz=-0.15 -0.40 1.45 rpy=0 0 3.14 -> xyz=0.02 0.3 0.2 rpy=0.0 3.14 0.0; parent base_link -> base_camera
- joint scan_joint: origin xyz=0 -0.17 1.57 rpy=0 0 0 -> xyz=0.25 -0.15 1.57 rpy=0 0 0

File: src/robile_robot/urdf/save.urdf (robot description, URDF)
Before this commit: robot ugv_robot, 7 links, 6 joints
Links:
- link base_link: geometry collision mesh filename=package://robile_robot/models/body5.stl; visual mesh filename=package://robile_robot/models/body5.stl
Joints:
- added joint base_to_ur5_base: type fixed, parent base_link, child ur5_base_link, origin xyz=-0.15 -0.1 1.12 rpy=0 0 1.57
- joint camera_joint: origin xyz=0 0 1.45 rpy=0 0 3.14 -> xyz=-0.15 -0.40 1.45 rpy=0 0 3.14

File: src/robile_robot/xacro/robile_robot_ur5.xacro (robot description, xacro)
@@ -2,6 +2,5 @@
 <robot xmlns:xacro="http://ros.org/wiki/xacro" name="mobile_robot">
 <xacro:include filename="$(find ur_description)/urdf/inc/ur5_macro.xacro"/>
-<xacro:include filename="$(find ur_description)/urdf/inc/ur3_macro.xacro"/>
-    <!-- Thân -->
+  <!-- Thân -->
   <link name="base_link">
     <visual>
@@ -21,21 +20,15 @@
     <inertial>
       <mass value="2"/>
-      <inertia ixx="0.4465" ixy="0" ixz="0" iyy="0.3468" iyz="0.0" izz="0.4026"/>
-    </inertial>
-  </link>
-<joint name="base_to_ur3_base" type="fixed">
-    <parent link="base_link"/>
-    <child link="ur3_base_link"/>  <!-- Kiểm tra lại tên của link này trong UR5 -->
-    <origin xyz="0.1 -0.8 0.7" rpy="3.14 1.57 1.57"/>
-  </joint>
-<joint name="base_to_ur5_base" type="fixed">
+      <inertia ixx="0.4465" ixy="0" ixz="0" iyy="0.3468" iyz="0.0" izz="0.4465"/>
+    </inertial>
+  </link>
+  <joint name="base_to_ur5_base" type="fixed">
     <parent link="base_link"/>
     <child link="ur5_base_link"/>  <!-- Kiểm tra lại tên của link này trong UR5 -->
-    <origin xyz="0.1 0.5 0.7" rpy="0 1.57 1.57"/>
+    <origin xyz="-0.15 -0.1 1.12" rpy="0 0 1.57"/>
   </joint>
   <!-- Include UR5 -->
   <xacro:ur5_robot prefix="ur5_"/>
-  <xacro:ur5_robot prefix="ur3_"/>
-<!-- Bánh xe -->
+  <!-- Bánh xe -->
   <link name="wheel_ph_trc">
     <visual>
@@ -140,6 +133,6 @@
         <publishWheelJointState>true</publishWheelJointState>
         <!-- Wheel Dynamics -->
-        <wheelAcceleration>200.0</wheelAcceleration>
-        <wheelTorque>200.0</wheelTorque>
+        <wheelAcceleration>50.0</wheelAcceleration>
+        <wheelTorque>50.0</wheelTorque>
         <updateRate>100</updateRate>
         <rosDebugLevel>na</rosDebugLevel>
@@ -173,21 +166,39 @@
   <!-- <camera> -->
 <!-- Base Camera -->
-<link name="camera_link">
+<link name="base_camera">
         <visual>
             <geometry>
-                <mesh filename="package://robile_robot/models/eye.stl" scale="0.5 0.5 0.5"/>
+                <mesh filename="package://robile_robot/models/eye4.stl"/>
             </geometry>
-            <origin xyz="-1.3 -0.8 -1.55" rpy="1.57 0 1.57"/>
+            <origin xyz="0 0 0" rpy="1.57 0 1.57"/>
         </visual>
         <inertial>
-            <mass value="0.1"/>
-            <inertia ixx="0.00004167" ixy="0.000" ixz="0.00" iyy="0.00007083" iyz="0.0" izz="0.00010417"/>
+            <mass value="0.4"/>
+            <inertia ixx="0.03867" ixy="0.000" ixz="0.00" iyy="0.013667" iyz="0.0" izz="0.04167"/>
         </inertial>
     </link>
+    <link name="camera_link">
+    <visual>
+      <geometry>
+        <cylinder radius="0.07" length="0.05"/>
+      </geometry>
+      <origin xyz="0.0 0.0 0.0" rpy="0.0 -1.57 0.0"/>
+      </visual>
+      <inertial>
+        <mass value="0.2"/>
+        <inertia ixx="0.00028667" ixy="0.000" ixz="0.00" iyy="0.00028667" iyz="0.0" izz="0.00049"/>
+      </inertial>
+    </link>
     <!-- Camera Joint -->
+    <joint name="base_camera_joint" type="fixed">
+        <parent link="base_link"/>
+        <child link="base_camera"/>
+        <origin xyz="0 -0.65 1.115" rpy="0 0 0"/>
+    </joint>
     <joint name="camera_joint" type="fixed">
-        <parent link="base_link"/>
-        <child link="camera_link"/>
-        <origin xyz="-0.15 -0.40 1.45" rpy="0 0 3.14"/>
+      <origin xyz="0.02 0.3 0.2" rpy="0.0 3.14 0.0"/>
+      <parent link="base_camera"/>
+      <child link="camera_link"/>
+      <axis xyz="0.0 0.0 0.0"/>
     </joint>
   <!-- Camera Work -->
@@ -195,5 +206,5 @@
         <material>Gazebo/Red</material>
         <sensor name="camera" type="camera">
-            <pose> 1.25 -0.4 2 0 0 0 </pose>
+            <pose> 0 0 0 1.57 0 0 </pose>
             <visualize>true</visualize>
             <update_rate>10</update_rate>
@@ -215,5 +226,5 @@
         </sensor>
     </gazebo>
-  <!-- Base Sensor -->
+    <!-- Base Sensor -->
   <link name="base_scan">
     <visual>
@@ -244,5 +255,5 @@
     <parent link="base_link"/>
     <child link="base_scan"/>
-    <origin xyz="0 -0.17 1.57" rpy="0 0 0"/>
+    <origin xyz="0.25 -0.15 1.57" rpy="0 0 0"/>
   </joint>
 <!-- Sensor Work -->
